Commit message: - Added the camera arm link to the terabot discription

File: terabot_description/urdf/terabot.xacro (robot description, xacro)
@@ -137,4 +137,11 @@
       <material name="Blue"/>
     </visual>
+     <visual>
+      <origin xyz="${(-100.49/2)*BASE+wrist_pitch_link_x_offset} ${230.1*BASE-(229/2)*BASE+wrist_pitch_link_y_offset} 0" rpy="0 ${PI/2} 0" />
+      <geometry>
+        <mesh filename="package://terabot_description/meshes/arm_camera.stl" scale="0.001 0.001 0.001"/>
+      </geometry>
+      <material name="red"/>
+    </visual>
     <collision>
       <geometry>

Commit message: - Modified terabot model links and joints orientation

File: terabot_description/urdf/terabot.xacro (robot description, xacro)
@@ -28,7 +28,7 @@
   </link>
   <joint name="shoulder_joint" type="revolute">
-    <origin xyz="0 0 ${(80)*BASE}"/>
-    <axis xyz="0 0 1"/>
-    <limit effort="1000.0" lower="${-170*(PI/180)}" upper="${170*(PI/180)}" velocity="0.5"/>
+    <origin xyz="0 0 ${(80)*BASE}" rpy="0 0 ${-pi}"/>
+    <axis xyz="0 0 1"/>
+    <limit effort="1000.0" lower="${170*(PI/180)}" upper="${-170*(PI/180)}" velocity="0.5"/>
     <parent link="arm_base_link"/>
     <child link="shoulder_link"/>
@@ -37,4 +37,11 @@
   <link name="shoulder_link">
     <visual>
+      <origin xyz="0 0 ${-(80/2)*BASE}" rpy="0 ${-pi/2} ${-pi/2}" />
+      <geometry>
+        <mesh filename="package://terabot_description/meshes/shoulder.stl" scale="0.001 0.001 0.001"/>
+      </geometry>
+      <material name="Blue"/>
+    </visual>
+    <collision>
       <origin xyz="0 0 ${-(80/2)*BASE}" rpy="0 ${-pi/2} ${pi/2}" />
       <geometry>
@@ -42,11 +49,4 @@
       </geometry>
       <material name="Blue"/>
-    </visual>
-    <collision>
-      <origin xyz="0 0 ${-(80/2)*BASE}" rpy="0 ${-pi/2} ${pi/2}" />
-      <geometry>
-        <mesh filename="package://terabot_description/meshes/shoulder.stl" scale="0.001 0.001 0.001"/>
-      </geometry>
-      <material name="Blue"/>
     </collision>
     <inertial>
@@ -60,7 +60,7 @@
   </link>
   <joint name="forearm_joint" type="revolute">
-    <origin xyz="0 0 ${(229/2)*BASE}" rpy="${PI/2} 0 0"/>
-    <axis xyz="0 0 1"/>
-    <limit effort="1000.0" lower="${-35*(PI/180)}" upper="${90*(PI/180)}" velocity="0.5"/>
+    <origin xyz="0 0 ${(229/2)*BASE}" rpy="${PI/2} ${-PI/2} ${-PI}"/>
+    <axis xyz="0 0 1"/>
+    <limit effort="1000.0" lower="${-90*(PI/180)}" upper="${0*(PI/180)}" velocity="0.5"/>
     <parent link="shoulder_link"/>
     <child link="forearm_link"/>
@@ -92,5 +92,5 @@
   </link>
   <joint name="upper_arm_joint" type="revolute">
-    <origin xyz="${419.1*BASE} 0 0"/>
+    <origin xyz="${419.1*BASE} 0 0" rpy="0 0 0"/>
     <axis xyz="0 0 1"/>
     <limit effort="1000.0" lower="${-170*(PI/180)}" upper="${162*(PI/180)}" velocity="0.5"/>

Commit message: -fixed some color issues

File: terabot_description/urdf/terabot.xacro (robot description, xacro)
@@ -10,5 +10,5 @@
         <mesh filename="package://terabot_description/meshes/base.stl" scale="0.001 0.001 0.001"/>
       </geometry>
-      <material name="Gray"/>
+      <material name="orange"/>
     </visual>
     <collision>
@@ -41,5 +41,5 @@
         <mesh filename="package://terabot_description/meshes/shoulder.stl" scale="0.001 0.001 0.001"/>
       </geometry>
-      <material name="Blue"/>
+      <material name="orange"/>
     </visual>
     <collision>
@@ -48,5 +48,5 @@
         <mesh filename="package://terabot_description/meshes/shoulder.stl" scale="0.001 0.001 0.001"/>
       </geometry>
-      <material name="Blue"/>
+      <material name="orange"/>
     </collision>
     <inertial>
@@ -73,5 +73,5 @@
         <mesh filename="package://terabot_description/meshes/forearm.stl" scale="0.001 0.001 0.001"/>
       </geometry>
-      <material name="Blue"/>
+      <material name="orange"/>
     </visual>
     <collision>
@@ -80,5 +80,5 @@
         <mesh filename="package://terabot_description/meshes/forearm.stl" scale="0.001 0.001 0.001"/>
       </geometry>
-      <material name="Blue"/>
+      <material name="orange"/>
     </collision>
     <inertial>
@@ -105,5 +105,5 @@
         <mesh filename="package://terabot_description/meshes/upper_arm.stl" scale="0.001 0.001 0.001"/>
       </geometry>
-      <material name="Blue"/>
+      <material name="orange"/>
     </visual>
     <collision>
@@ -135,5 +135,5 @@
         <mesh filename="package://terabot_description/meshes/wrist_pitch.stl" scale="0.001 0.001 0.001"/>
       </geometry>
-      <material name="Blue"/>
+      <material name="orange"/>
     </visual>
      <visual>
@@ -142,5 +142,5 @@
         <mesh filename="package://terabot_description/meshes/arm_camera.stl" scale="0.001 0.001 0.001"/>
       </geometry>
-      <material name="red"/>
+      <material name="orange"/>
     </visual>
     <collision>
@@ -172,5 +172,5 @@
         <mesh filename="package://terabot_description/meshes/wrist_roll.stl" scale="0.001 0.001 0.001"/>
       </geometry>
-      <material name="black"/>
+      <material name="orange"/>
     </visual>
     <inertial>
@@ -196,5 +196,5 @@
         <mesh filename="package://terabot_description/meshes/left_finger.stl" scale="0.001 0.001 0.001"/>
       </geometry>
-      <material name="Grey"/>
+      <material name="red"/>
     </visual>
     <inertial>
@@ -221,5 +221,5 @@
         <mesh filename="package://terabot_description/meshes/right_finger.stl" scale="0.001 0.001 0.001"/>
       </geometry>
-      <material name="Grey"/>
+      <material name="red"/>
     </visual>
     <inertial>

Commit message: - The range is wong! It

File: terabot_description/urdf/terabot.xacro (robot description, xacro)
@@ -30,5 +30,5 @@
     <origin xyz="0 0 ${(80)*BASE}" rpy="0 0 ${-pi}"/>
     <axis xyz="0 0 1"/>
-    <limit effort="1000.0" lower="${170*(PI/180)}" upper="${-170*(PI/180)}" velocity="0.5"/>
+    <limit effort="1000.0" lower="${-170*(PI/180)}" upper="${170*(PI/180)}" velocity="0.5"/>
     <parent link="arm_base_link"/>
     <child link="shoulder_link"/>

Commit message: - Changed the color of the gripper

File: terabot_description/urdf/terabot.xacro (robot description, xacro)
@@ -196,5 +196,5 @@
         <mesh filename="package://terabot_description/meshes/left_finger.stl" scale="0.001 0.001 0.001"/>
       </geometry>
-      <material name="red"/>
+      <material name="brown"/>
     </visual>
     <inertial>
@@ -221,5 +221,5 @@
         <mesh filename="package://terabot_description/meshes/right_finger.stl" scale="0.001 0.001 0.001"/>
       </geometry>
-      <material name="red"/>
+      <material name="brown"/>
     </visual>
     <inertial>

Commit message: - Modification done for camera_arm calibration

File: terabot_description/urdf/terabot.xacro (robot description, xacro)
@@ -158,9 +158,31 @@
     </inertial>
   </link>
+ <!-- added end effector for calibration -->
+ <joint name="end_effector_joint" type="fixed">
+   <origin xyz="0.09 ${wrist_roll_joint_z_offset} 0" rpy="0 0 0"/> <!-- original is 0.085 but we have the torque sensor...-->
+      <axis xyz="0 0 1"/>
+      <parent link="wrist_pitch_link"/>
+      <child link="end_effector"/>
+      <dynamics damping="100.0" friction="100.0" />
+      </joint>
+      <!-- end_effector -->
+      <link name="end_effector">
+	<origin xyz="0 0 0" rpy="0 0 0"/>
+      <inertial>
+      <origin xyz="0 0 1" rpy="0 0 0"/>
+      <mass value="0.01"/>
+      <inertia
+      ixx="1.0" ixy="0.0" ixz="0.0"
+      iyy="1.0" iyz="0.0"
+      izz="1.0"/>
+      </inertial>
+      </link>
+ <!-- modified the following part to add end_effector link (marker) for calibration -->
  <joint name="wrist_roll_joint" type="revolute">
-    <origin xyz="${50*BASE+0.013+wrist_roll_joint_x_offset} ${wrist_roll_joint_z_offset} 0" rpy="0 ${PI/2} 0"/>
+    <!-- origin xyz="${50*BASE+0.013+wrist_roll_joint_x_offset} ${wrist_roll_joint_z_offset} 0" rpy="0 ${PI/2} 0"/ -->
+     <origin xyz="0.07 0 0" rpy="0 ${PI/2} 0"/>
     <axis xyz="0 0 1"/>
     <limit effort="1000.0" lower="${-170*(PI/180)}" upper="${170*(PI/180)}" velocity="0.5"/>
-    <parent link="wrist_pitch_link"/>
+    <parent link="end_effector"/>
     <child link="wrist_roll_link"/>
     <dynamics damping="0.7"/>

Commit message: - Added missing tags and transmissions for the gripper

File: terabot_description/urdf/terabot.xacro (robot description, xacro)
@@ -256,7 +256,9 @@
   <transmission name="tran1">
     <type>transmission_interface/SimpleTransmission</type>
-    <joint name="shoulder_joint"/>
+    <joint name="shoulder_joint">
+      <hardwareInterface>PositionJointInterface</hardwareInterface>
+    </joint>
     <actuator name="motor1">
-      <hardwareInterface>EffortJointInterface</hardwareInterface>
+        <hardwareInterface>PositionJointInterface</hardwareInterface>
       <mechanicalReduction>1</mechanicalReduction>
     </actuator>
@@ -264,7 +266,9 @@
   <transmission name="tran2">
     <type>transmission_interface/SimpleTransmission</type>
-    <joint name="forearm_joint"/>
+    <joint name="forearm_joint">
+        <hardwareInterface>PositionJointInterface</hardwareInterface>
+    </joint>
     <actuator name="motor2">
-      <hardwareInterface>EffortJointInterface</hardwareInterface>
+        <hardwareInterface>PositionJointInterface</hardwareInterface>
       <mechanicalReduction>1</mechanicalReduction>
     </actuator>
@@ -272,7 +276,9 @@
   <transmission name="tran3">
     <type>transmission_interface/SimpleTransmission</type>
-    <joint name="upper_arm_joint"/>
+    <joint name="upper_arm_joint">
+        <hardwareInterface>PositionJointInterface</hardwareInterface>
+    </joint>
     <actuator name="motor3">
-      <hardwareInterface>EffortJointInterface</hardwareInterface>
+        <hardwareInterface>PositionJointInterface</hardwareInterface>
       <mechanicalReduction>1</mechanicalReduction>
     </actuator>
@@ -280,7 +286,9 @@
   <transmission name="tran4">
     <type>transmission_interface/SimpleTransmission</type>
-    <joint name="wrist_pitch_joint"/>
+    <joint name="wrist_pitch_joint">
+        <hardwareInterface>PositionJointInterface</hardwareInterface>
+    </joint>
     <actuator name="motor4">
-      <hardwareInterface>EffortJointInterface</hardwareInterface>
+        <hardwareInterface>PositionJointInterface</hardwareInterface>
       <mechanicalReduction>1</mechanicalReduction>
     </actuator>
@@ -288,9 +296,31 @@
   <transmission name="tran5">
     <type>transmission_interface/SimpleTransmission</type>
-    <joint name="wrist_roll_joint"/>
+    <joint name="wrist_roll_joint">
+        <hardwareInterface>PositionJointInterface</hardwareInterface>
+    </joint>
     <actuator name="motor5">
-      <hardwareInterface>EffortJointInterface</hardwareInterface>
-      <mechanicalReduction>1</mechanicalReduction>
-    </actuator>
+        <hardwareInterface>PositionJointInterface</hardwareInterface>
+      <mechanicalReduction>1</mechanicalReduction>
+    </actuator>
+  </transmission>
+  <transmission name="tran6">
+      <type>transmission_interface/SimpleTransmission</type>
+      <joint name="gripper_r_finger_joint">
+          <hardwareInterface>PositionJointInterface</hardwareInterface>
+      </joint>
+      <actuator name="motor6">
+          <hardwareInterface>PositionJointInterface</hardwareInterface>
+          <mechanicalReduction>1</mechanicalReduction>
+      </actuator>
+  </transmission>
+  <transmission name="tran7">
+      <type>transmission_interface/SimpleTransmission</type>
+      <joint name="gripper_l_finger_joint">
+          <hardwareInterface>PositionJointInterface</hardwareInterface>
+      </joint>
+      <actuator name="motor7">
+          <hardwareInterface>PositionJointInterface</hardwareInterface>
+          <mechanicalReduction>1</mechanicalReduction>
+      </actuator>
   </transmission>
 </robot>

Commit message: - Modification for adding the gripper part to the hardware interface

File: terabot_description/urdf/terabot.xacro (robot description, xacro)
@@ -207,5 +207,5 @@
   <joint name="gripper_l_finger_joint" type="revolute">
     <origin xyz="${gripper_l_finger_joint_x_offset} 0 -0.0145" rpy="0 ${3*PI/2} ${3*PI/2}"/>
-    <limit effort="1000.0" lower="0.0" upper="${115*(PI/180)}" velocity="0.5"/>
+    <limit effort="1000.0" lower="0.0" upper="${40*(PI/180)}" velocity="0.5"/>
     <axis xyz="0 0 -1"/>
     <parent link="wrist_roll_link"/>
@@ -231,5 +231,5 @@
    <joint name="gripper_r_finger_joint" type="revolute">
     <origin xyz="${gripper_r_finger_joint_x_offset} 0 -0.0145" rpy="0 ${3*PI/2} ${3*PI/2}"/>
-    <limit effort="1000.0" lower="0.0" upper="${115*(PI/180)}" velocity="0.5"/>
+    <limit effort="1000.0" lower="0.0" upper="${40*(PI/180)}" velocity="0.5"/>
     <axis xyz="0 0 1"/>
     <mimic joint="gripper_l_finger_joint"/>

Commit message: - Modifications

File: terabot_description/urdf/terabot.xacro (robot description, xacro)
@@ -107,9 +107,9 @@
       <material name="orange"/>
     </visual>
-    <collision>
+<!--    <collision>
       <geometry>
         <cylinder length="${364.49*BASE}" radius="0.05"/>
       </geometry>
-    </collision>
+    </collision>-->
     <inertial>
       <origin xyz="0 0 0" rpy="0 0 0"/>
@@ -144,9 +144,9 @@
       <material name="orange"/>
     </visual>
-    <collision>
+<!--    <collision>
       <geometry>
         <cylinder length="${364.49*BASE}" radius="0.05"/>
       </geometry>
-    </collision>
+    </collision>-->
     <inertial>
       <origin xyz="0 0 0" rpy="0 0 0"/>

Commit message: -trial

File: terabot_description/urdf/terabot.xacro (robot description, xacro)
@@ -160,5 +160,6 @@
  <!-- added end effector for calibration -->
  <joint name="end_effector_joint" type="fixed">
-   <origin xyz="0.09 ${wrist_roll_joint_z_offset} 0" rpy="0 0 0"/> <!-- original is 0.085 but we have the torque sensor...-->
+      <origin xyz="0.09 ${wrist_roll_joint_z_offset} 0" rpy="0 0 0"/>    <!-- before modifications -->
+<!--   <origin xyz="0.09 0.04 0.006" rpy="0 0 0"/> --><!-- original is 0.085 but we have the torque sensor...-->
       <axis xyz="0 0 1"/>
       <parent link="wrist_pitch_link"/>
@@ -180,6 +181,7 @@
  <!-- modified the following part to add end_effector link (marker) for calibration -->
  <joint name="wrist_roll_joint" type="revolute">
-    <!-- origin xyz="${50*BASE+0.013+wrist_roll_joint_x_offset} ${wrist_roll_joint_z_offset} 0" rpy="0 ${PI/2} 0"/ -->
-     <origin xyz="0.07 0 0" rpy="0 ${PI/2} 0"/>
+   <!-- origin xyz="${50*BASE+0.013+wrist_roll_joint_x_offset} ${wrist_roll_joint_z_offset} 0" rpy="0 ${PI/2} 0"/ --> <!-- when the parent is wrist pitch joint -->
+        <origin xyz="0.07 0 0" rpy="0 ${PI/2} 0"/><!-- when the end effector is the parent -->
+  <!--   <origin xyz="0.07 -0.005 0" rpy="0 ${PI/2} 0"/>-->
     <axis xyz="0 0 1"/>
     <limit effort="1000.0" lower="${-170*(PI/180)}" upper="${170*(PI/180)}" velocity="0.5"/>
@@ -190,5 +192,7 @@
   <link name="wrist_roll_link">
     <visual>
-      <origin xyz="-0.0322 ${0.4*BASE+wrist_roll_link_y_offset} ${-18.5*BASE+wrist_roll_link_x_offset}" rpy="0 -${PI} ${3*PI/2}" />
+<!--      <origin xyz="-0.0322 ${0.4*BASE+wrist_roll_link_y_offset} ${-18.5*BASE+wrist_roll_link_x_offset}" rpy="0 -${PI} ${3*PI/2}" />--><!-- when the parent is wrist pitch joint -->
+<origin xyz="-0.0322 ${0.4*BASE+wrist_roll_link_y_offset} ${-18.5*BASE+wrist_roll_link_x_offset}" rpy="0 -${PI} ${3*PI/2}" /><!-- when the end effector is the parent -->
+<!--     <origin xyz="-0.0315 0 ${-18.5*BASE+wrist_roll_link_x_offset}" rpy="0 -${PI} ${3*PI/2}" />    -->
       <geometry>
         <mesh filename="package://terabot_description/meshes/wrist_roll.stl" scale="0.001 0.001 0.001"/>
